File: rev_a/hdw/Thermal_Camera/Mechanical.kicad_sch (KiCad schematic)
At the start: 0 parts

Commit message: copied lots of circuitry to reuse
Parts:
- added H? (x8): MountingHole, MountingHole:MountingHole_3mm, symbol Mechanical:MountingHole
