File: rev_a/hdw/Thermal_Camera/Mechanical.kicad_sch (KiCad schematic)
At the start: 8 parts

Commit message: blah blah
Parts:
- removed H? (x4): MountingHole, MountingHole:MountingHole_3mm, symbol Mechanical:MountingHole
