File: rev_a/hdw/Thermal_Camera/Status_LEDs.kicad_sch (KiCad schematic)
At the start: 20 parts

Commit message: assigned some part numbers
Parts:
- C? (x4): Digi-Key PN (none) -> 490-10697-1-ND
- D?: Digi-Key PN (none) -> 1497-1219-1-ND
- D? (x3): Digi-Key PN (none) -> VLMS1500-GS08CT-ND
Changed lines of the file:
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@@
 			)
 		)
-		(property "Digi-Key PN" ""
+		(property "Digi-Key PN" "490-10697-1-ND"
 			(at 96.52 67.31 0)
 			(effects
@@
 			)
 		)
-		(property "Digi-Key PN" ""
+		(property "Digi-Key PN" "1497-1219-1-ND"
 			(at 234.188 171.069 0)
 			(effects
@@
 			)
 		)
-		(property "Digi-Key PN" ""
+		(property "Digi-Key PN" "490-10697-1-ND"
 			(at 45.72 67.31 0)
 			(effects
@@
 			)
 		)
-		(property "Digi-Key PN" ""
+		(property "Digi-Key PN" "490-10697-1-ND"
 			(at 45.72 16.51 0)
 			(effects
@@
 			)
 		)
-		(property "Digi-Key PN" ""
+		(property "Digi-Key PN" "VLMS1500-GS08CT-ND"
 			(at 73.66 90.805 0)
 			(effects
@@
 			)
 		)
-		(property "Digi-Key PN" ""
+		(property "Digi-Key PN" "VLMS1500-GS08CT-ND"
 			(at 124.46 90.805 0)
 			(effects
@@
 			)
 		)
-		(property "Digi-Key PN" ""
+		(property "Digi-Key PN" "VLMS1500-GS08CT-ND"
 			(at 124.46 40.005 0)
 			(effects
@@
 			)
 		)
-		(property "Digi-Key PN" ""
+		(property "Digi-Key PN" "490-10697-1-ND"
 			(at 96.52 16.51 0)
 			(effects
