File: rev_a/hdw/Thermal_Camera/Status_LEDs.kicad_sch (KiCad schematic)
At the start: 20 parts

Commit message: assigned resistor part numbers
Parts:
- R? (x4): Digi-Key PN (none) -> RMCF0402FT10K0CT-ND
- R? (x4): Digi-Key PN (none) -> RMCF0402FT1K00CT-ND
Changed lines of the file:
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@@
 			)
 		)
-		(property "Digi-Key PN" ""
+		(property "Digi-Key PN" "RMCF0402FT10K0CT-ND"
 			(at 95.885 103.505 0)
 			(effects
@@
 			)
 		)
-		(property "Digi-Key PN" ""
+		(property "Digi-Key PN" "RMCF0402FT1K00CT-ND"
 			(at 66.04 22.225 0)
 			(effects
@@
 			)
 		)
-		(property "Digi-Key PN" ""
+		(property "Digi-Key PN" "RMCF0402FT10K0CT-ND"
 			(at 95.885 41.275 0)
 			(effects
@@
 			)
 		)
-		(property "Digi-Key PN" ""
+		(property "Digi-Key PN" "RMCF0402FT1K00CT-ND"
 			(at 116.84 22.225 0)
 			(effects
@@
 			)
 		)
-		(property "Digi-Key PN" ""
+		(property "Digi-Key PN" "RMCF0402FT10K0CT-ND"
 			(at 45.085 52.705 0)
 			(effects
@@
 			)
 		)
-		(property "Digi-Key PN" ""
+		(property "Digi-Key PN" "RMCF0402FT10K0CT-ND"
 			(at 45.085 103.505 0)
 			(effects
@@
 			)
 		)
-		(property "Digi-Key PN" ""
+		(property "Digi-Key PN" "RMCF0402FT1K00CT-ND"
 			(at 66.04 73.025 0)
 			(effects
@@
 			)
 		)
-		(property "Digi-Key PN" ""
+		(property "Digi-Key PN" "RMCF0402FT1K00CT-ND"
 			(at 116.84 73.025 0)
 			(effects
