File: rev_a/hdw/Thermal_Camera/Thermal_Camera.kicad_pcb (KiCad board)
At the start: 2 copper layers, 100 x 100 mm, 517 parts, among them J1401 18650 Holder, J1501 PICKIT4, J1502 MRST, J2001 Micro_SD_Card_Det_Hirose_DM3AT, J201 +12V IN, J2101 LCD Pixel Data, J2301 I2C, J2302 UART, J2303 VOSPI, J2304 FLASH SPI, J2601 USB_B_Mini, Q1401 DMN3042L, Q1402 DMN3042L, Q1501 BSS214NW, Q401 BSS214NW, Q402 ZXMS6004FFTA, Q601 BSS214NW, Q602 ZXMS6004FFTA, SW1501 MRST, SW2501 RESET, SW2901 Cap_Touch, SW2902 Cap_Touch, U1001 74LVC1G97, U1002 TPS7A92, U1101 INA231A, U1102 MCP9804, U1201 DIO5661CD6, U1301 INA231A, U1302 MCP9804, U1401 BQ27441DRZT-G1A, U1402 MAX8903G, U1403 BQ29700, U1601 74LVC1G97, U1701 PIC32MZ2064DAR176, U2001 SST25VF080B-50-4x-S2Ax, U2002 TPS22810DRV, U201 TPS26600RHFT, U2201 FT234XD, U2202 74LVC1G97, U2203 FXMA108, U2301 DS1683, U2302 MCP9804, U2401 FLIR_Lepton3p5_Socket, U2501 74LVC1G97, U2502 TPS3808G33, U2503 74LVC1G97, U2504 TUSB2046BIRHBT, U2601 TPS7A92, U2602 TPD3S044DBVR, U2701 74LVC1G97, U2702 74LVC1G97, U2703 74LVC1G97, U2704 74LVC1G97, U2705 74LVC1G97, U2706 74LVC1G97, U2707 74LVC1G97, U2801 74LVC1G97, U2802 74LVC1G97, U2803 74LVC1G97, U2804 74LVC1G97, U2901 AT42QT1010-TSHR, U2902 AT42QT1010-TSHR, U2903 74LVC1G97, U2904 74LVC1G97, U301 INA231A, U302 MCP9804, U401 74LVC1G97, U402 TPS62130A, U501 INA231A, U502 MCP9804, U601 74LVC1G97, U602 TPS62130A, U701 INA231A, U702 MCP9804, U801 TPS7A92, U901 INA231A, U902 MCP9804, X1601 ECS-2520MV-240-BN, X1602 ECS-327KE, X2401 ECS-2520MV-250-CN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

Commit message: placed battery charger circuitry
Parts:
- C1402, C1404, C1405, C1406, C1407, C1410, C1411, C1412, C2607, C301, C302, C303, L1401, R1401, R1403, R1404, R1405, R1406, R1408, R1409, R1410, R1411, R1413, U1402, U301, U302: moved to B.Cu
- R1414, R1415, U1403: moved to F.Cu
- moved R1415 417.3 mm to (88.4, 49.0), turned to -90 degrees
- moved TH1401 406.5 mm to (101.8, 58.1)
- moved TH1402 403.8 mm to (102.8, 58.1)
- moved Q1402 354.4 mm to (156.5, 47.1), turned to -90 degrees
- moved Q1401 352.8 mm to (156.5, 51.0), turned to 90 degrees
- moved C1414 350.2 mm to (159.7, 44.5), turned to 180 degrees
- moved U1403 350.1 mm to (159.5, 46.4), turned to 90 degrees
- moved R1414 349.8 mm to (157.7, 44.5)
- moved C2501 342.8 mm to (42.1, 120.9)
- moved C2502 342.8 mm to (47.4, 115.4)
- moved C2503 342.8 mm to (42.1, 121.8)
- moved C2504 342.8 mm to (50.4, 120.0)
- moved C2505 342.8 mm to (50.4, 121.0)
- moved C2506 342.8 mm to (46.9, 120.9)
- moved C2507 342.8 mm to (43.4, 124.7)
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Other:
- board text added: "+3.0V"
- board text removed: "+3.3V"

Commit message: placed some power supplies
Parts:
- C2401, C2402, C2403, C2404, C2405, C2901, C2902, C2903, C2904, C2905, C2906, C2907, C2908, C401, C403, C601, C603, D401, D601, L2401, Q401, Q402, Q601, Q602, R2401, R2404, R2406, R2408, R2409, R2410, R2411, R2412, R2413, R2414, R2415, R2905, R2906, R2909, R2910, R401, R402, R404, R405, R407, R601, R602, R604, R605, R607, X2401: moved to F.Cu
- C404, C405, C406, C407, C604, C605, C606, C607, L401, L601, R2402, R2403, R2405, R2407, R2907, R2908, R403, R406, R408, R409, R603, R606, R608, R609, TP401, TP601, U2401, U2901, U2902, U2903, U2904, U401, U402, U601, U602: moved to B.Cu
- moved C2201 332.6 mm to (74.6, 161.9)
- moved R2201 332.6 mm to (72.2, 164.4)
- moved R2203 332.6 mm to (72.6, 158.8)
- moved U2201 332.6 mm to (71.1, 161.7)
- moved U2203 332.6 mm to (81.9, 162.3)
- moved C2202 332.6 mm to (81.4, 160.6)
- moved C2203 332.6 mm to (67.6, 162.4)
- moved C2204 332.6 mm to (85.6, 163.9)
- moved C2205 332.6 mm to (80.5, 160.6)
- moved C2206 332.6 mm to (67.6, 163.3)
- moved C2207 332.6 mm to (67.6, 161.5)
- moved C2208 332.6 mm to (71.6, 158.8)
- moved C2209 332.6 mm to (70.7, 158.8)
- moved C2210 332.6 mm to (82.4, 160.6)
- moved C2211 332.6 mm to (83.3, 160.6)
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
Commit message: placed more power supplies
Parts:
- C1002, C1003, C1005, C1006, C1101, C1102, C801, C802, C804, C805, C901, C902, R1005, R1007, R1008, R804, R806, R807, TP1001, TP801, U1002, U1101, U801, U901: moved to B.Cu
- C1004, C803, R1004, R1006, R803, R805: moved to F.Cu
- moved R803 328.6 mm to (109.0, 92.8), turned to -90 degrees
- moved R804 327.8 mm to (109.5, 93.9), turned to 0 degrees
- moved R805 326.5 mm to (110.1, 92.8), turned to -90 degrees
- moved C803 323.5 mm to (111.2, 95.1), turned to -90 degrees
- moved R802 322.5 mm to (112.4, 96.6), turned to 0 degrees
- moved C801 322.5 mm to (112.3, 91.4), turned to 0 degrees
- moved C802 322.5 mm to (112.3, 92.3), turned to 0 degrees
- moved U801 320.4 mm to (113.3, 94.5), turned to 180 degrees
- moved R801 319.3 mm to (114.1, 96.6), turned to 0 degrees
- moved C804 318.3 mm to (114.4, 92.3), turned to 180 degrees
- moved C805 318.3 mm to (114.4, 91.4), turned to 180 degrees
- moved R806 315.4 mm to (115.9, 94.2)
- moved R807 315.4 mm to (115.9, 95.9)
- moved TP801 313.3 mm to (117.0, 92.0), turned to 180 degrees
- moved C1002 297.4 mm to (136.6, 95.5)
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
Commit message: placed LCD backlight driver
Parts:
- C1001, C1201, C2501, C2502, C2503, C2509, R1003, R2503, R2504, R2505: moved to F.Cu
- C1303, C2504, C2505, C2506, C2507, C2508, L2501, R2501, R2502, R2506, R2507, U1001, U1302, U2501, U2502, U2503, U2504, X2501: moved to B.Cu
- moved L1201 306.2 mm to (136.3, 137.9), turned to 180 degrees
- moved D1201 302.4 mm to (133.1, 132.7), turned to -90 degrees
- moved R1201 301.9 mm to (137.5, 135.9), turned to 0 degrees
- moved C1204 300.8 mm to (135.3, 132.7), turned to -90 degrees
- moved U1201 299.4 mm to (137.7, 133.2), turned to -90 degrees
- moved C1202 298.9 mm to (139.5, 133.9), turned to 90 degrees
- moved R1204 298.8 mm to (131.0, 129.7)
- moved R1205 298.8 mm to (130.4, 130.4)
- moved R1206 298.8 mm to (129.9, 129.7)
- moved C1203 297.3 mm to (134.5, 129.3), turned to 0 degrees
- moved C1201 296.3 mm to (141.1, 132.7), turned to 90 degrees
- moved R1202 296.0 mm to (138.8, 130.9), turned to 0 degrees
- moved R1203 294.7 mm to (138.8, 129.9), turned to 0 degrees
- moved C1001 290.4 mm to (139.8, 89.0), turned to 0 degrees
- moved R1003 290.4 mm to (139.8, 90.0), turned to 0 degrees
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