File: rev_a/hdw/Thermal_Camera/LCD_Backlight_Telemetry.kicad_sch (KiCad schematic)
At the start: 7 parts, among them U1301 INA231A

Commit message: assigned some part numbers
Parts:
- C? (x3): Digi-Key PN (none) -> 490-10697-1-ND
Changed lines of the file:
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@@
 			)
 		)
-		(property "Digi-Key PN" ""
+		(property "Digi-Key PN" "490-10697-1-ND"
 			(at 113.03 52.07 0)
 			(effects
@@
 			)
 		)
-		(property "Digi-Key PN" ""
+		(property "Digi-Key PN" "490-10697-1-ND"
 			(at 135.89 76.2 0)
 			(effects
@@
 			)
 		)
-		(property "Digi-Key PN" ""
+		(property "Digi-Key PN" "490-10697-1-ND"
 			(at 135.89 144.78 0)
 			(effects
