File: rev_a/hdw/Thermal_Camera/Thermal_Camera.kicad_sch (KiCad schematic)
At the start: 0 parts

Commit message: lots of schematic progress
Other:
- added sheet Capacitive Touch (Capacitive_Touch.kicad_sch)
- note added: "29. Capacitive Touch"
- note added: "30. Mechanical"
- note removed: "29. Mechanical"
- note removed: "Add capacitive touch"
Changed lines of the file:
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@@
 	(title_block
 		(title "Thermal Camera")
-		(date "2023-12-07")
+		(date "2024-05-24")
 		(rev "PRELIM")
 		(company "Drew Maatman and Michael Laffin")
@@
 		)
 	)
+	(text "29. Capacitive Touch"
+		(exclude_from_sim no)
+		(at 193.04 77.47 0)
+		(effects
+			(font
+				(face "Courier New")
+				(size 2.032 2.032)
+				(thickness 0.508)
+				(bold yes)
+			)
+			(justify left bottom)
+		)
+	)
 	(text "13. LCD Backlight Telemetry"
 		(exclude_from_sim no)
@@
 		)
 	)
-	(text "Add capacitive touch"
-		(exclude_from_sim no)
-		(at 38.1 183.134 0)
-		(effects
-			(font
-				(size 5.08 5.08)
-				(thickness 1.016)
-				(bold yes)
-				(color 194 0 0 1)
-			)
-			(justify left bottom)
-		)
-	)
 	(text "17. PIC32MZ DA Power"
 		(exclude_from_sim no)
@@
 		)
 	)
-	(text "29. Mechanical"
-		(exclude_from_sim no)
-		(at 193.04 77.47 0)
+	(text "30. Mechanical"
+		(exclude_from_sim no)
+		(at 193.04 87.63 0)
 		(effects
 			(font
@@
 	)
 	(sheet
+		(at 234.95 73.66)
+		(size 12.7 3.81)
+		(fields_autoplaced yes)
+		(stroke
+			(width 0.1524)
+			(type solid)
+		)
+		(fill
+			(color 0 0 0 0.0000)
+		)
+		(property "Sheetname" "Capacitive Touch"
+			(at 234.95 72.9484 0)
+			(effects
+				(font
+					(size 1.27 1.27)
+				)
+				(justify left bottom)
+			)
+		)
+		(property "Sheetfile" "Capacitive_Touch.kicad_sch"
+			(at 234.95 78.0546 0)
+			(effects
+				(font
+					(size 1.27 1.27)
+				)
+				(justify left top)
+				(hide yes)
+			)
+		)
+		(instances
+			(project "Thermal_Camera"
+				(path "/4bd21e0b-5408-4b93-866e-c82ac5b31fa9"
+					(page "29")
+				)
+			)
+		)
+	)
+	(sheet
 		(at 72.39 83.82)
 		(size 12.7 3.81)
@@
 	)
 	(sheet
-		(at 234.95 73.66)
+		(at 234.95 83.82)
 		(size 12.7 3.81)
 		(fields_autoplaced yes)
@@
 		)
 		(property "Sheetname" "Mechanical"
-			(at 234.95 72.9484 0)
+			(at 234.95 83.1084 0)
 			(effects
 				(font
@@
 		)
 		(property "Sheetfile" "Mechanical.kicad_sch"
-			(at 234.95 78.0546 0)
-			(effects
-				(font
-					(size 1.27 1.27)
-				)
-				(justify left top)
-				(hide yes)
-			)
-		)
-		(instances
-			(project "Thermal_Camera"
-				(path "/4bd21e0b-5408-4b93-866e-c82ac5b31fa9"
-					(page "29")
+			(at 234.95 88.2146 0)
+			(effects
+				(font
+					(size 1.27 1.27)
+				)
+				(justify left top)
+				(hide yes)
+			)
+		)
+		(instances
+			(project "Thermal_Camera"
+				(path "/4bd21e0b-5408-4b93-866e-c82ac5b31fa9"
+					(page "30")
 				)
 			)
@@
 				)
 				(justify left top)
-			)
-		)
+				(hide yes)
+			)
+		)

Commit message: added some stitching caps
Other:
- added sheet Stitching Caps (stitching_caps.kicad_sch)
- note added: "31. Stitching Caps"
Changed lines of the file:
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@@
 	(title_block
 		(title "Thermal Camera")
-		(date "2024-05-24")
-		(rev "PRELIM")
+		(date "2024-09-20")
+		(rev "A")
 		(company "Drew Maatman and Michael Laffin")
 	)
@@
 		)
 	)
+	(text "31. Stitching Caps"
+		(exclude_from_sim no)
+		(at 193.04 97.79 0)
+		(effects
+			(font
+				(face "Courier New")
+				(size 2.032 2.032)
+				(thickness 0.508)
+				(bold yes)
+			)
+			(justify left bottom)
+		)
+	)
 	(text "21. Graphic LCD"
 		(exclude_from_sim no)
@@
 				)
 			)
+		)
+	)
+	(sheet
+		(at 234.95 93.98)
+		(size 12.7 3.81)
+		(fields_autoplaced yes)
+		(stroke
+			(width 0.1524)
+			(type solid)
+		)
+		(fill
+			(color 0 0 0 0.0000)
+		)
+		(property "Sheetname" "Stitching Caps"
+			(at 234.95 93.2684 0)
+			(effects
+				(font
+					(size 1.27 1.27)
+				)
+				(justify left bottom)
+			)
+		)
+		(property "Sheetfile" "stitching_caps.kicad_sch"
+			(at 234.95 98.3746 0)
+			(effects
+				(font
+					(size 1.27 1.27)
+				)
+				(justify left top)
+				(hide yes)
+			)
+		)
+		(instances
+			(project "Thermal_Camera"
+				(path "/4bd21e0b-5408-4b93-866e-c82ac5b31fa9"
+					(page "31")
+				)
+			)
